File: PCB/Previous versions/Street_Fighter_v1.1.brd (EAGLE design)
At the start: 53.3 x 77.5 mm, 42 parts, among them Q1 BSS138, Q2 BSS138, Q3 FQP30N06L, Q4 BSS138, U1 ARDUINO_YUN_SHIELDYUN, U2 MCP6231RT-E/OT

Commit message: Fixes Issue #2 and Issue #4. New XBee socket + SPI
Parts:
- removed UVD: Maxbotix 1320, SparkFun-Connectors:1X04
- added C3, C8: 10uF, SparkFun-Capacitors:1206
- added C4: 0.1uF, SparkFun-Capacitors:1206
- added J1: FEMALE 2x3, SparkFun-Connectors:2X3
- added PIR1: MOTION, SparkFun-Connectors:1X03
- added Q10, Q5, Q6, Q7, Q8, Q9: BSS138, SparkFun-DiscreteSemi:SOT23
- added R10, R11, R14, R15, R19, R20, R21, R22, R23, R24, R25, R26, R27: 4.7K, SparkFun-Passives:1206
- added SJ1, SJ2: (no value), SparkFun-Retired:SJ_3_PASTE1&2
- added U3: (no value), SparkFun-PowerIC:SOT223
- added XBEE1: XBEE-2B3, SparkFun-RF:XBEE-SMD
- R1, R12, R13, R2, R3, R4: value 10K -> 4.7K
- T-ROAD: value MLX90614-ACF? -> MLX90614-ACF
- moved R9 1.27 mm to (41.9, 14.6)
- renumbered TEMP to DS18B20
Connections:
- net XB-AD3 renamed XB-SS
- removed net LIDAR-CTRL: LIDAR.5
- removed net RANGE-ANALOG: U1.A1, UVD.3
- removed net RANGE-CTRL: UVD.2
- new net 3V3: U1.3V3
- new net MISO: J1.1
- new net MOSI: J1.4
- new net N$3: SJ1.2
- new net N$5: SJ2.2
- new net RST: J1.5
- new net RX-XB2: Q10.3, R27.1, U1.11
- new net SCK: J1.3
- new net SONAR-PULSEIN: PIR1.2, U1.A0
- new net TX-XB2: Q9.3, R25.1, U1.12
- new net XB-ATTN: XBEE.19
- new net XB-CLK: XBEE.18
- new net XB-MISO: XBEE.4
- new net XB-MOSI: XBEE.11
- new net XB2-DIN: Q9.2, R24.1, XBEE1.3
- new net XB2-DOUT: Q10.2, R26.1, XBEE1.2
- new net XB2-RSSI: XBEE1.6
- net +3V3: now also C3.2, C4.2, Q10.1, Q5.1, Q6.1, Q7.1, Q8.1, Q9.1, R11.2, R15.2, R20.2, R22.2, R24.2, R26.2, U3.2, U3.4, XBEE1.1; no longer U1.3V3
- net +5V: now also C8.2, J1.2, PIR1.3, R10.2, R14.2, R19.2, R21.2, R23.2, R25.2, R27.2, U3.3; no longer UVD.4
- net GND: now also C3.1, C4.1, C8.1, J1.6, PIR1.1, U3.1, XBEE1.10; no longer UVD.1
- net TEMP: now also R10.1
- net TX-XB: now also Q5.3, Q6.3, Q7.3, Q8.3, R14.1, R19.1, R21.1, R23.1
- net XB-SLEEP3V: now also XBEE1.13
- net XB-TX3V: now also Q5.2, Q6.2, Q7.2, Q8.2, R11.1, R15.1, R20.1, R22.1
Routing:
- net +5V: track 172.0 -> 0.00 mm, vias 2 -> 0
- net +3V3: track 124.1 -> 0.00 mm, vias 4 -> 0
- net TX-XB: track 47.9 -> 0.00 mm, vias 2 -> 0
- net XB-SLEEP: track 43.5 -> 0.00 mm, vias 2 -> 0
- net LED-CONTROL: track 42.5 -> 0.00 mm
- net RX-XB: track 41.6 -> 0.00 mm, vias 2 -> 0
- net N$4: track 30.0 -> 0.00 mm, vias 1 -> 0
- net SDA: track 27.1 -> 0.00 mm, vias 1 -> 0
- net SCL: track 26.8 -> 0.00 mm
- net SCL@1: track 23.7 -> 0.00 mm
- net N$2: track 22.9 -> 0.00 mm
- net LIDAR-PWM: track 22.1 -> 0.00 mm
- net XB-TX3V: track 21.5 -> 0.00 mm
- net XB-RX3V: track 20.6 -> 0.00 mm, vias 2 -> 0
- net XB-RTS: track 19.9 -> 0.00 mm
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Other:
- board text removed: "MISO"
- board text removed: "MOSI"
- board text removed: "SCK"
- board text removed: "SS"
