File: PCB/Street_Fighter_v1.3.sch (EAGLE design)
At the start: 72 parts, among them J1 FEMALE 2x3, Q1 BSS138, Q10 BSS138, Q2 BSS138, Q3 FQP30N06L, Q4 BSS138, Q5 BSS138, Q6 BSS138, Q7 BSS138, Q9 BSS138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

Commit message: StreetFighter v1.3 board - Fixed bad pin assignments for SoftSerial
Parts:
- added SPARE: A1, SparkFun-Connectors:M03PTH
- XBEE-IN, XBEE-OUT: value (none) -> JUMPER-PAD-3-2OF3_NC_BY_TRACE_SMALL; device SparkFun-Retired:SOLDERJUMPER_2WAYS -> SparkFun-Passives:JUMPER-PAD-3-2OF3_NC_BY_TRACE_SMALL
Connections:
- net RX-XB renamed SPI-ATTN
- net TX-XB renamed SPI-SS
- net XB-SCK renamed 3V-SCK
- removed net XB-RX3V: Q2.S, R3.1, XBEE-OUT.2
- removed net XB-TX3V: Q1.S, R1.1, XBEE-IN.2
- new net 3V-MISO: Q5.S, R11.1, XBEE-OUT.2
- new net 3V-MOSI: Q6.S, R15.1, XBEE-IN.2
- new net SPARE: SPARE.2, U1.A1
- net +5V: now also SPARE.3
- net GND: now also SPARE.1
- net LIDAR-PWM: now also U1.D12*; no longer U1.D10*
- net TX-XB2: now also U1.D10*; no longer U1.D12*
- net XB-ATTN: now also Q2.S, R3.1; no longer XBEE-OUT.1
- net XB-MISO: now also XBEE-OUT.1; no longer Q5.S, R11.1
- net XB-MOSI: now also XBEE-IN.1; no longer Q6.S, R15.1
- net XB-SS: now also Q1.S, R1.1; no longer XBEE-IN.1
Other:
- note added: "Spare"
- note removed: "Base Components"
- moved on the sheet: C1, CURRENT, Q10, Q4, Q5, Q6, Q7, Q9, R11, R12, R13, R14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
